File: hardware/Multipurpose Flight Computer.kicad_sch (KiCad schematic)
At the start: 0 parts

Commit message: Importing STM32 parts
Parts:
- added C1: 1uF, symbol Device:C
- added C2, C3, C5: 10uF, symbol Device:C
- added C4: 47nF, symbol Device:C
- added C6: 44uF, symbol Device:C
- added Card1: TF-01A, easyeda2kicad:TF-SMD_TF-01A, symbol easyeda2kicad:TF-01A
- added D1: LED, symbol Device:LED
- added J1: Screw_Terminal_01x02, symbol Connector:Screw_Terminal_01x02
- added L5: DFE252012F-1ROM=P2, symbol Device:L
- added R1, R2: 5.1K, symbol Device:R
- added R10, R11, R6, R7, R8, R9: 10K, symbol Device:R
- added R3: 3B3, symbol Device:R
- added R4: 5.23K, symbol Device:R
- added R5: 30.1K, symbol Device:R
- added U1: BMP580, easyeda2kicad:LGA-10_L2.0-W2.0-P0.50-TL_BMP580, symbol easyeda2kicad:BMP580
- added U1: BQ25883RGER, easyeda2kicad:VFQFPN-24_L4.0-W4.0-P0.50-BL-EP2.8, symbol easyeda2kicad:BQ25883RGER
- added U3: ICM-45686, easyeda2kicad:LGA-14_L3.0-W2.5-P0.50-TL, symbol easyeda2kicad:ICM-45686
- added U4: TPS63070RNMR, easyeda2kicad:VQFN-15_L3.0-W2.5-P0.50-BL, symbol easyeda2kicad:TPS63070RNMR
- added U5: STM32F722RETx, Package_QFP:LQFP-64_10x10mm_P0.5mm, symbol MCU_ST_STM32F7:STM32F722RETx
- added U6: LMR51430, Package_TO_SOT_SMD:SOT-23-6, symbol Regulator_Switching:LMR51430
- added USB1: TYPE-C 16PIN 2MD, easyeda2kicad:USB-C-SMD_TYPE-C-16PIN-2MD-073, symbol easyeda2kicad:TYPE-C16PIN2MD
Connections:
- new net: D1.2 (A), R7.2
- new net: R4.2, R5.1, R6.1, U1.7 (TS)
- new net: R1.1, USB1.A5 (CC1)
- new net: USB1.A6 (Dp1), USB1.B6 (Dp2)
- new net: R2.1, USB1.B5 (CC2)
- new net: R3.1, U1.8 (ILIM)
- new net: C5.1, L5.1, U1.21 (PMID), U1.22 (PMID)
- new net: C4.2, U1.12 (BTST)
- new net: D1.1 (K), U1.2 (STAT)
- new net: U5.18 (VSS), U5.31 (VSS), U5.47 (VSS), U5.63 (VSS)
- new net +3.3V: R10.1, R11.1, R7.1, R8.1, R9.1
- new net BAT+: C2.1, J1.1 (Pin_1), U1.13 (BAT), U1.14 (BAT)
- new net BQ_CE: U1.3 (~{CE})
- new net BQ_INT: R11.2, U1.6 (~{INT})
- new net BQ_PG: R8.2, U1.9 (~{PG})
- new net BTST: C4.1, L5.2, U1.17 (SW), U1.18 (SW)
- new net GND: C1.2, C2.2, C3.2, C5.2, C6.2, J1.2 (Pin_2), R1.2, R2.2, R3.2, R5.2, R6.2, U1.19 (GND), U1.20 (GND), U1.25 (EP), USB1.13 (EH), USB1.14 (EH), USB1.A1B12 (GND), USB1.B1A12 (GND)
- new net I2C_SCL: R10.2, U1.5 (SCL)
- new net I2C_SDA: R9.2, U1.4 (SDA)
- new net USB_DN: USB1.A7 (Dn1), USB1.B7 (Dn2)
- new net VBUS: C1.1, U1.23 (VBUS), USB1.A4B9 (VBUS), USB1.B4A9 (VBUS)
- new net VREGN: C3.1, R4.1, U1.11 (REGN)
- new net VSYS: C6.1, U1.15 (SYS), U1.16 (SYS)
- no-connect marks 0 -> 5

Commit message: Assigning Footprints
Parts:
- added C10, C11, C13, C17, C18: 22uF, symbol Device:C
- added C12, C7, C8, C9: 10uF, symbol Device:C
- added C14, C15, C19, C20, C21, C22, C23, C24, C25, C26, C27, C37: 100nF, symbol Device:C
- added C16, C32: 2.2uF, symbol Device:C
- added C28, C29, C30, C31: 1uF, symbol Device:C
- added C33, C34: 20pF, symbol Device:C
- added C35, C36: 6.8pF, symbol Device:C
- added J2, J3: Conn_01x03, symbol Connector_Generic:Conn_01x03
- added L2: 1.5uH, symbol Device:L
- added L3: 5.6uH, symbol Device:L
- added L4: FCM1608KF-601T03, easyeda2kicad:L0603, symbol easyeda2kicad:FCM1608KF-601T03
- added R12, R13, R16, R17, R18, R19, R21, R22, R30: 10K, Resistor_SMD:R_0201_0603Metric, symbol Device:R
- added R14: 100K, Resistor_SMD:R_0402_1005Metric, symbol Device:R
- added R15: 22.1K, Resistor_SMD:R_0201_0603Metric, symbol Device:R
- added SW1, SW2: TS-1088-AR02016, easyeda2kicad:SW-SMD_L3.9-W3.0-P4.45, symbol easyeda2kicad:TS-1088-AR02016
- added X1: X322525MOB4SI, easyeda2kicad:CRYSTAL-SMD_4P-L3.2-W2.5-BL, symbol easyeda2kicad:X322525MOB4SI
- added X2: Q13FC1350000400, easyeda2kicad:FC-135R_L3.2-W1.5, symbol easyeda2kicad:Q13FC1350000400
- J1: footprint (none) -> TerminalBlock:TerminalBlock_Xinya_XY308-2.54-2P_1x02_P2.54mm_Horizontal
- L1: renamed from L5; value DFE252012F-1ROM=P2 -> 1uH
- R1, R10, R11, R2, R3, R4, R5, R6, R7, R8, R9: footprint (none) -> Resistor_SMD:R_0201_0603Metric
- renumbered U3 to U2, U5 to U3, U1 to U4, U4 to U5
Connections:
- net +3.3V: now also Card1.4 (VDD), U2.5 (VDDIO), U2.8 (VDD), U3.1 (VBAT), U3.19 (VDD), U3.32 (VDD), U3.48 (VDD), U3.64 (VDD), U4.1 (VDDIO), U4.10 (VDD), C17.1, C18.1, C19.1, C20.1, C21.1, C22.1, C23.1, C24.1, C25.1, C26.1, C27.1, C28.1, C29.1, C30.1, C31.1, L3.2, L4.1, R14.1, R16.1, R17.1, R18.1, R19.1, R21.1, R30.1, SW2.1
- net BQ_CE: now also U3.61 (PB8)
- net BQ_INT: now also U3.57 (PB5)
- net GND: now also Card1.10 (GND), Card1.11 (GND), Card1.12 (GND), Card1.13 (GND), Card1.6 (VSS), U2.6 (GND), U3.12 (VSSA), U3.18 (VSS), U3.31 (VSS), U3.47 (VSS), U3.63 (VSS), U4.3 (VSS), U4.5 (SDO), U4.6 (CSB), U4.8 (VSS), U4.9 (VSS), U5.10 (PGND), U5.15 (Vsel), U5.4 (GND), U5.6 (FB2), U6.1 (GND), C10.2, C11.2, C12.2, C13.2, C14.2, C16.2, C17.2, C18.2, C19.2, C20.2, C21.2, C22.2, C23.2, C24.2, C25.2, C26.2, C27.2, C28.2, C29.2, C30.2, C31.2, C32.2, C33.2, C34.2, C35.2, C36.2, C37.2, C7.2, C8.2, C9.2, J2.3 (Pin_3), J3.3 (Pin_3), R15.2, R22.2, SW1.1, X1.2 (GND), X1.4 (GND)
- net I2C_SCL: now also U3.58 (PB6), U4.2 (SCK)
- net I2C_SDA: now also U3.59 (PB7), U4.4 (SDI)
- net USB_DN: now also U3.44 (PA11)
- net VSYS: now also U5.12 (Vin), U6.3 (VIN), U6.5 (EN), C16.1, C7.1, C8.1, C9.1, R12.2
- net at USB1.A6 (Dp1), USB1.B6 (Dp2): now also U3.45 (PA12)
- net at U5.1 (PS/SYNC): now also U5.14 (EN), R12.1
- net at U5.11 (L1): now also L2.2
- net at U5.2 (PG): now also R13.1
- net at U5.3 (Vaux): now also C14.1
- net +5V: now reaches U5.5 (FB)
- net +5V: now also U5.7 (Vout), C10.1, C11.1, C12.1, C13.1, J2.1 (Pin_1), J3.1 (Pin_1), R13.2
- net at U5.9 (L2): now also L2.1
- net BMP_INT: now reaches U4.7 (INT)
- net BMP_INT: now also U3.62 (PB9)
- net SD_DAT2: now reaches Card1.1 (DAT2(RSV))
- net SD_DAT2: now also U3.51 (PC10), R18.2
- net SD_DAT3: now reaches Card1.2 (CDDAT3(CS))
- net SD_DAT3: now also U3.52 (PC11), R19.2
- net SD_CMD: now reaches Card1.3 (CMD(DI))
- net SD_CMD: now also U3.54 (PD2), R30.2
- net SD_CLK: now reaches Card1.5 (CLK(SCLK))
- net SD_CLK: now also U3.53 (PC12), R21.2
- net SD_DAT0: now reaches Card1.7 (DAT0(D0))
- net SD_DAT0: now also U3.39 (PC8), R16.2
- net SD_DAT1: now reaches Card1.8 (DAT1(RSV))
- net SD_DAT1: now also U3.40 (PC9), R17.2
- net SD_CD: now reaches Card1.9 (CD)
- net SD_CD: now also U3.55 (PB3)
- net at U6.2 (SW): now also C15.2, L3.1
- net at U6.4 (FB): now also R14.2, R15.1
- net at U6.6 (CB): now also C15.1
- net ICO_SD0: now reaches U2.1 (AP_SDO/AP_AD0)
- net ICM_CS: now reaches U2.12 (AP_CS)
- net ICM_CS: now also U3.20 (PA4)
- net ICM_SDK: now reaches U2.13 (AP_SCL/AP_SCLK)
- net ICM_SDI: now reaches U2.14 (AP_SDA/AP_SDIO/AP_SDI)
- net ICO_INT1: now reaches U2.4 (INT1/INT)
- net ICM_INT2: now reaches U2.9 (INT2/FSYNC/CLKIN)
- net ICM_INT2: now also U3.25 (PB0), U3.42 (PA9)
- net at U3.13 (VDDA): now also L4.2
- net SERVO1: now reaches U3.14 (PA0)
- net SERVO1: now also J2.2 (Pin_2), J3.2 (Pin_2)
- net SERVO2: now reaches U3.15 (PA1)
- net ICM_SCK: now reaches U3.21 (PA5)
- net ICM_SD0: now reaches U3.22 (PA6)
- net ICM_SD1: now reaches U3.23 (PA7)
- net ICM_INT1: now reaches U3.24 (PC4)
- net ICM_INT1: now also U3.41 (PA8)
- net LSE_IN: now reaches U3.3 (PC14)
- net LSE_IN: now also C35.1, X2.1
- net at U3.30 (VCAP_1): now also C32.1
- net LSE_OUT: now reaches U3.4 (PC15)
- net LSE_OUT: now also C36.1, X2.2
- net HSE_IN: now reaches U3.5 (PH0)
- net HSE_IN: now also C33.1, X1.1 (OSC1)
- net HSE_OUT: now reaches U3.6 (PH1)
- net HSE_OUT: now also C34.1, X1.3 (OSC2)
- net BOOT: now reaches U3.60 (BOOT0)
- net BOOT: now also R22.1, SW2.2
- net RESET: now reaches U3.7 (NRST)
- net RESET: now also C37.1, SW1.2
- no-connect marks 5 -> 32
Other:
- note added: "3.3V Buck"
- note added: "5V Buck-Boost"
- note added: "Battery Charger"
- note added: "Buttons"
- note added: "Crystals"
- note added: "Decoupling"
- note added: "IMU"
- note added: "MicroSD Card"
- note added: "Pressure Sensor"
- note added: "STM32"
- note added: "Servos"
- note added: "USB-C"
- moved on the sheet: C1, C2, C3, C4, C5, C6, Card1, D1, J1, L1, R1, R10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

Commit message: drc
Parts:
- C1, C17, C18, C28, C29, C3, C30, C31, C5: footprint (none) -> Capacitor_SMD:C_0402_1005Metric
- C10, C11, C13, C7, C8: footprint (none) -> Capacitor_SMD:C_0805_2012Metric
- C12, C16, C2, C6, C9: footprint (none) -> Capacitor_SMD:C_0603_1608Metric
- C14, C15, C19, C20, C21, C22, C23, C24, C25, C26, C27, C32, C33, C34, C35, C36, C37, C4: footprint (none) -> Capacitor_SMD:C_0201_0603Metric
- D1: footprint (none) -> LED_SMD:LED_0402_1005Metric
- J2, J3: footprint (none) -> Connector_PinHeader_2.54mm:PinHeader_1x03_P2.54mm_Vertical
- L1: footprint (none) -> easyeda2kicad:L2520
- L2: footprint (none) -> easyeda2kicad:IND-SMD_L4.0-W4.0-A
- L3: footprint (none) -> easyeda2kicad:IND-SMD_L3.0-W3.0
- R15: footprint Resistor_SMD:R_0201_0603Metric -> Resistor_SMD:R_0402_1005Metric
Connections:
- net ICM_SDI is gone; now on net ICM_SD1: U2.14 (AP_SDA/AP_SDIO/AP_SDI)
- net ICM_SDK is gone; now on net ICM_SCK: U2.13 (AP_SCL/AP_SCLK)
- net ICO_INT1 is gone; now on net ICM_INT1: U2.4 (INT1/INT)
- net ICO_SD0 is gone; now on net ICM_SD0: U2.1 (AP_SDO/AP_AD0)
- net SERVO1: no longer J3.2 (Pin_2)
- net SERVO2: now also J3.2 (Pin_2)
- net USB_DP: now reaches U3.45 (PA12), USB1.A6 (Dp1), USB1.B6 (Dp2)
Changed lines of the file:
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@@
 	(wire
 		(pts
-			(xy 46.99 46.99) (xy 57.15 46.99)
-		)
-		(stroke
-			(width 0)
-			(type default)
-		)
-	)
-	(wire
-		(pts
 			(xy 38.1 160.02) (xy 38.1 161.29)
 		)
@@
 	(wire
 		(pts
-			(xy 46.99 41.91) (xy 57.15 41.91)
-		)
-		(stroke
-			(width 0)
-			(type default)
-		)
-	)
-	(wire
-		(pts
 			(xy 337.82 95.25) (xy 331.47 95.25)
 		)
@@
 		)
 	)
-	(label "USB_DP"
-		(at 57.15 41.91 180)
-		(effects
-			(font
-				(size 1.27 1.27)
-			)
-			(justify right bottom)
-		)
-	)
 	(label "SD_CD"
 		(at 245.11 162.56 180)
@@
 		)
 	)
+	(label "USB_DP"
+		(at 46.99 41.91 0)
+		(effects
+			(font
+				(size 1.27 1.27)
+			)
+			(justify left bottom)
+		)
+	)
 	(label "BQ_CE"
 		(at 245.11 175.26 180)
@@
 		)
 	)
-	(label "ICO_INT1"
+	(label "ICM_INT1"
 		(at 148.59 256.54 0)
 		(effects
@@
 	)
 	(label "USB_DP"
-		(at 57.15 46.99 180)
+		(at 46.99 46.99 0)
 		(effects
 			(font
 				(size 1.27 1.27)
 			)
-			(justify right bottom)
+			(justify left bottom)
 		)
 	)
@@
 		)
 	)
-	(label ""
-		(at 57.15 41.91 180)
-		(effects
-			(font
-				(size 1.27 1.27)
-			)
-			(justify right bottom)
-		)
-	)
 	(label "VBUS"
 		(at 57.15 54.61 180)
@@
 		)
 	)
-	(label "ICO_SD0"
+	(label "ICM_SD0"
 		(at 148.59 248.92 0)
 		(effects
@@
 		)
 	)
-	(label "SERVO1"
+	(label "SERVO2"
 		(at 370.84 52.07 0)
 		(effects
@@
 		)
 	)
-	(label "ICM_SDK"
+	(label "ICM_SCK"
 		(at 281.94 251.46 180)
 		(effects
@@
 		)
 	)
-	(label "ICM_SDI"
+	(label "ICM_SD1"
 		(at 281.94 248.92 180)
 		(effects
@@
 			)
 		)
-		(property "Footprint" ""
+		(property "Footprint" "Capacitor_SMD:C_0805_2012Metric"
 			(at 369.2652 203.2 0)
 			(effects
@@
 			)
 		)
-		(property "Footprint" ""
+		(property "Footprint" "Capacitor_SMD:C_0201_0603Metric"
 			(at 177.4952 35.56 0)
 			(effects
@@
 			)
 		)
-		(property "Footprint" ""
+		(property "Footprint" "Capacitor_SMD:C_0805_2012Metric"
 			(at 379.4252 203.2 0)
 			(effects
@@
 			)
 		)
-		(property "Footprint" ""
+		(property "Footprint" "Capacitor_SMD:C_0201_0603Metric"
 			(at 192.7352 35.56 0)
 			(effects
@@
 			)
 		)
-		(property "Footprint" ""
+		(property "Footprint" "Capacitor_SMD:C_0201_0603Metric"
 			(at 169.8752 35.56 0)
 			(effects
@@
 			)
 		)
-		(property "Footprint" "Resistor_SMD:R_0201_0603Metric"
+		(property "Footprint" "Resistor_SMD:R_0402_1005Metric"
 			(at 85.852 251.46 90)
 			(effects
@@
 			)
 		)
-		(property "Footprint" ""
+		(property "Footprint" "Capacitor_SMD:C_0201_0603Metric"
 			(at 287.9852 273.05 0)
 			(effects
@@
 			)
 		)
-		(property "Footprint" ""
+		(property "Footprint" "easyeda2kicad:IND-SMD_L4.0-W4.0-A"
 			(at 323.85 201.93 0)
 			(effects
@@
 			)
 		)
-		(property "Footprint" ""
+		(property "Footprint" "Capacitor_SMD:C_0402_1005Metric"
 			(at 111.4552 140.97 0)
 			(effects
@@
 			)
 		)
-		(property "Footprint" ""
+		(property "Footprint" "Capacitor_SMD:C_0201_0603Metric"
 			(at 130.5052 63.5 0)
 			(effects
@@
 			)
 		)
-		(property "Footprint" ""
+		(property "Footprint" "Capacitor_SMD:C_0201_0603Metric"
 			(at 364.49 184.4548 0)
 			(effects
@@
 			)
 		)
-		(property "Footprint" ""
+		(property "Footprint" "Capacitor_SMD:C_0805_2012Metric"
 			(at 303.2252 193.04 0)
 			(effects
@@
 			)
 		)
-		(property "Footprint" ""
+		(property "Footprint" "Capacitor_SMD:C_0603_1608Metric"
 			(at 72.0852 105.41 0)
 			(effects
@@
 			)
 		)
-		(property "Footprint" ""
+		(property "Footprint" "Capacitor_SMD:C_0201_0603Metric"
 			(at 115.2652 63.5 0)
 			(effects
@@
 			)
 		)
-		(property "Footprint" ""
+		(property "Footprint" "Capacitor_SMD:C_0201_0603Metric"
 			(at 140.6652 266.7 0)
 			(effects
@@
 			)
 		)
-		(property "Footprint" ""
+		(property "Footprint" "Capacitor_SMD:C_0201_0603Metric"
 			(at 72.0852 240.03 0)
 			(effects
@@
 			)
 		)
-		(property "Footprint" ""
+		(property "Footprint" "Capacitor_SMD:C_0402_1005Metric"
 			(at 174.9552 58.42 0)
 			(effects
@@
 			)
 		)
-		(property "Footprint" ""
+		(property "Footprint" "Capacitor_SMD:C_0805_2012Metric"
 			(at 312.1152 193.04 0)
 			(effects
@@
 			)
 		)
-		(property "Footprint" ""
+		(property "Footprint" "Capacitor_SMD:C_0201_0603Metric"
 			(at 236.22 37.7952 0)
 			(effects
@@
 			)
 		)
-		(property "Footprint" ""
+		(property "Footprint" "Capacitor_SMD:C_0805_2012Metric"
 			(at 388.3152 203.2 0)
 			(effects
@@
 			)
 		)
-		(property "Footprint" ""
+		(property "Footprint" "Capacitor_SMD:C_0402_1005Metric"
 			(at 41.6052 148.59 0)
 			(effects
@@
 			)
 		)
-		(property "Footprint" ""
+		(property "Footprint" "easyeda2kicad:IND-SMD_L3.0-W3.0"
 			(at 81.28 240.03 0)
 			(effects
@@
 			)
 		)
-		(property "Footprint" ""
+		(property "Footprint" "Capacitor_SMD:C_0402_1005Metric"
 			(at 188.9252 58.42 0)
 			(effects
@@
 			)
 		)
-		(property "Footprint" ""
+		(property "Footprint" "Capacitor_SMD:C_0201_0603Metric"
 			(at 185.1152 35.56 0)
 			(effects
@@
 			)
 		)
-		(property "Footprint" ""
+		(property "Footprint" "Capacitor_SMD:C_0603_1608Metric"
 			(at 83.5152 114.3 0)
 			(effects
@@
 			)
 		)
-		(property "Footprint" ""
+		(property "Footprint" "Capacitor_SMD:C_0402_1005Metric"
 			(at 195.2752 58.42 0)
 			(effects
@@
 			)
 		)
-		(property "Footprint" ""
+		(property "Footprint" "Capacitor_SMD:C_0402_1005Metric"
 			(at 102.5652 247.65 0)
 			(effects
@@
 			)
 		)
-		(property "Footprint" ""
+		(property "Footprint" "Connector_PinHeader_2.54mm:PinHeader_1x03_P2.54mm_Vertical"
 			(at 387.35 33.02 0)
 			(effects
@@
 			)
 		)
-		(property "Footprint" ""
+		(property "Footprint" "Capacitor_SMD:C_0201_0603Metric"
 			(at 200.3552 35.56 0)
 			(effects
@@
 			)
 		)
-		(property "Footprint" ""
+		(property "Footprint" "Capacitor_SMD:C_0402_1005Metric"
 			(at 92.4052 247.65 0)
 			(effects
@@
 			)
 		)
-		(property "Footprint" ""
+		(property "Footprint" "easyeda2kicad:L2520"
 			(at 46.99 114.3 0)
 			(effects
@@
 			)
 		)
-		(property "Footprint" ""
+		(property "Footprint" "Capacitor_SMD:C_0201_0603Metric"
 			(at 110.1852 43.18 0)
 			(effects
@@
 			)
 		)
-		(property "Footprint" ""
+		(property "Footprint" "Capacitor_SMD:C_0201_0603Metric"
 			(at 343.8652 50.8 0)
 			(effects
@@
 			)
 		)
-		(property "Footprint" ""
+		(property "Footprint" "Capacitor_SMD:C_0603_1608Metric"
 			(at 321.0052 193.04 0)
 			(effects
@@
 			)
 		)
-		(property "Footprint" ""
+		(property "Footprint" "Capacitor_SMD:C_0201_0603Metric"
 			(at 187.6552 185.42 0)
 			(effects
@@
 			)
 		)
-		(property "Footprint" ""
+		(property "Footprint" "Capacitor_SMD:C_0201_0603Metric"
 			(at 135.5852 38.1 0)
 			(effects
@@
 			)
 		)
-		(property "Footprint" ""
+		(property "Footprint" "Capacitor_SMD:C_0402_1005Metric"
 			(at 181.3052 58.42 0)
 			(effects
@@
 			)
 		)
-		(property "Footprint" ""
+		(property "Footprint" "Capacitor_SMD:C_0603_1608Metric"
 			(at 359.1052 203.2 0)
 			(effects
@@
 			)
 		)
-		(property "Footprint" ""
+		(property "Footprint" "Connector_PinHeader_2.54mm:PinHeader_1x03_P2.54mm_Vertical"
 			(at 387.35 52.07 0)
 			(effects
@@
 			)
 		)
-		(property "Footprint" ""
+		(property "Footprint" "Capacitor_SMD:C_0201_0603Metric"
 			(at 89.8652 125.73 0)
 			(effects
@@
 			)
 		)
-		(property "Footprint" ""
+		(property "Footprint" "Capacitor_SMD:C_0603_1608Metric"
 			(at 40.3352 245.11 0)
 			(effects
@@
 			)
 		)
-		(property "Footprint" ""
+		(property "Footprint" "LED_SMD:LED_0402_1005Metric"
 			(at 59.69 160.02 0)
 			(effects
@@
 			)
 		)
-		(property "Footprint" ""
+		(property "Footprint" "Capacitor_SMD:C_0201_0603Metric"
 			(at 291.7952 50.8 0)
 			(effects
@@
 			)
 		)
-		(property "Footprint" ""
+		(property "Footprint" "Capacitor_SMD:C_0402_1005Metric"
 			(at 49.2252 127 0)
 			(effects

Commit message: Updating KiCad
Changed lines of the file:
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@@
 			(effects
 				(font
-					(size 1.016 1.016)
+					(size 1.27 1.27)
 				)
 				(justify left)
@@
 		(dnp no)
 		(property "Reference" "L3"
-			(at 81.788 236.982 90)
-			(effects
-				(font
-					(size 0.762 0.762)
+			(at 81.788 235.966 90)
+			(effects
+				(font
+					(size 1.27 1.27)
 				)
 			)
 		)
 		(property "Value" "5.6uH"
-			(at 82.55 238.506 90)
-			(effects
-				(font
-					(size 0.762 0.762)
-				)
-			)
+			(at 82.042 237.998 90)
+			(effects
+				(font
+					(size 1.27 1.27)
+				)
+			)

Commit message: Finishing Touches
Parts:
- added H1: MountingHole, MountingHole:MountingHole_2.2mm_M2_DIN965_Pad_TopBottom, symbol Mechanical:MountingHole
Changed lines of the file:
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@@
+	)
+	(symbol
+		(lib_id "Mechanical:MountingHole")
+		(at 335.28 238.76 0)
+		(unit 1)
+		(exclude_from_sim no)
+		(in_bom no)
+		(on_board yes)
+		(dnp no)
+		(fields_autoplaced yes)
+		(property "Reference" "H1"
+			(at 337.82 237.4899 0)
+			(effects
+				(font
+					(size 1.27 1.27)
+				)
+				(justify left)
+			)
+		)
+		(property "Value" "MountingHole"
+			(at 337.82 240.0299 0)
+			(effects
+				(font
+					(size 1.27 1.27)
+				)
+				(justify left)
+			)
+		)
+		(property "Footprint" "MountingHole:MountingHole_2.2mm_M2_DIN965_Pad_TopBottom"
+			(at 335.28 238.76 0)
+			(effects
+				(font
+					(size 1.27 1.27)
+				)
+				(hide yes)
+			)
+		)
+		(property "Datasheet" "~"
+			(at 335.28 238.76 0)
+			(effects
+				(font
+					(size 1.27 1.27)
+				)
+				(hide yes)
+			)
+		)
+		(property "Description" "Mounting Hole without connection"
+			(at 335.28 238.76 0)
+			(effects
+				(font
+					(size 1.27 1.27)
+				)
+				(hide yes)
+			)
+		)
+		(instances
+			(project ""
+				(path "/af0ac348-c8cb-4da6-83ea-ab1101947074"
+					(reference "H1")
+					(unit 1)
+				)
+			)
+		)
 	)
 	(symbol

Commit message: 4-layer upgrade
Parts:
- added C38: 100nF, Capacitor_SMD:C_0201_0603Metric, symbol Device:C
- added C39: 1uF, Capacitor_SMD:C_0402_1005Metric, symbol Device:C
Connections:
- net GND: now also C38.2, C39.2
- net at L4.2, U3.13 (VDDA): now also C38.1, C39.1
Other:
- moved on the sheet: L4

Commit message: Finalized Board Design
Parts:
- added U7: TPD4EUSB30, Package_SON:USON-10_2.5x1.0mm_P0.5mm, symbol Power_Protection:TPD4EUSB30
Connections:
- net GND: now also U7.3 (GND), U7.8 (GND)
- net USB_DN: now also U7.2 (D1-)
- net USB_DP: now also U7.1 (D1+)
- no-connect marks 32 -> 38
Other:
- moved on the sheet: R1, R2, USB1

Commit message: Bug Fixes
Parts:
- removed C20: 100nF, Capacitor_SMD:C_0201_0603Metric, symbol Device:C
- removed J1: Screw_Terminal_01x02, TerminalBlock:TerminalBlock_Xinya_XY308-2.54-2P_1x02_P2.54mm_Horizontal, symbol Connector:Screw_Terminal_01x02
- removed X2: Q13FC1350000400, easyeda2kicad:FC-135R_L3.2-W1.5, symbol easyeda2kicad:Q13FC1350000400
- added J4: Conn_01x02_Pin, easyeda2kicad:CONN-TH_XT30PW-M, symbol Connector:Conn_01x02_Pin
- added R20: 10K, Resistor_SMD:R_0201_0603Metric, symbol Device:R
- added R23: 4.7k, Resistor_SMD:R_0201_0603Metric, symbol Device:R
- C35: value 6.8pF -> 100nF
- C36: value 6.8pF -> 22uF; footprint Capacitor_SMD:C_0201_0603Metric -> Capacitor_SMD:C_0603_1608Metric
- C6: value 44uF -> 22uF
- C9: footprint Capacitor_SMD:C_0603_1608Metric -> Capacitor_SMD:C_0805_2012Metric
- R10, R9: value 10K -> 4.7k
- R3: value 3B3 -> 383; footprint Resistor_SMD:R_0201_0603Metric -> Resistor_SMD:R_0603_1608Metric
- R5: footprint Resistor_SMD:R_0201_0603Metric -> Resistor_SMD:R_0402_1005Metric
Connections:
- net +3.3V: now also C35.2, R20.2, R23.1
- net BAT+: now also J4.2 (Pin_2)
- net GND: now also C35.1, J4.1 (Pin_1); no longer C35.2, U4.6 (CSB)
- net ICM_CS: now also R20.1
- net USB_DN: now also U7.9 (NC)
- net USB_DP: now also U7.10 (NC)
- net VSYS: now also C36.1
- net LSE_IN: no longer names the net of U3.3 (PC14)
- net LSE_IN: no longer C35.1
- net LSE_OUT: no longer names the net of U3.4 (PC15)
- net LSE_OUT: no longer C36.1
- new net: R23.2, U4.6 (CSB)
