File: hardware/Multipurpose Flight Computer.kicad_sch (KiCad schematic)
At the start: 83 parts, among them J2 Conn_01x03, J3 Conn_01x03, J4 Conn_01x02_Pin, SW1 TS-1088-AR02016, SW2 TS-1088-AR02016, U1 BQ25883RGER, U2 ICM-45686, U3 STM32F722RETx, U4 BMP580, U5 TPS63070RNMR, U6 LMR51430, U7 TPD4EUSB30, X1 X322525MOB4SI

Commit message: Added software
Other:
- moved on the sheet: C33, C34, X1
Changed lines of the file:
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@@
 	(text "Crystals"
 		(exclude_from_sim no)
-		(at 121.158 16.764 0)
+		(at 124.714 17.018 0)
 		(effects
 			(font
@@
 	)
 	(junction
-		(at 134.62 30.48)
+		(at 138.43 36.83)
 		(diameter 0)
 		(color 0 0 0 0)
@@
 	)
 	(junction
-		(at 109.22 35.56)
+		(at 113.03 41.91)
 		(diameter 0)
 		(color 0 0 0 0)
@@
 	)
 	(junction
-		(at 109.22 44.45)
+		(at 113.03 50.8)
 		(diameter 0)
 		(color 0 0 0 0)
@@
 	)
 	(junction
-		(at 134.62 38.1)
+		(at 138.43 44.45)
 		(diameter 0)
 		(color 0 0 0 0)
@@
 	(wire
 		(pts
-			(xy 109.22 44.45) (xy 109.22 43.18)
+			(xy 113.03 50.8) (xy 113.03 49.53)
 		)
 		(stroke
@@
 	(wire
 		(pts
-			(xy 128.27 35.56) (xy 130.81 35.56)
+			(xy 132.08 41.91) (xy 134.62 41.91)
 		)
 		(stroke
@@
 	(wire
 		(pts
-			(xy 134.62 30.48) (xy 143.51 30.48)
+			(xy 138.43 36.83) (xy 147.32 36.83)
 		)
 		(stroke
@@
 	(wire
 		(pts
-			(xy 100.33 30.48) (xy 100.33 44.45)
+			(xy 104.14 36.83) (xy 104.14 50.8)
 		)
 		(stroke
@@
 	(wire
 		(pts
-			(xy 130.81 35.56) (xy 130.81 38.1)
+			(xy 134.62 41.91) (xy 134.62 44.45)
 		)
 		(stroke
@@
 	(wire
 		(pts
-			(xy 109.22 35.56) (xy 113.03 35.56)
+			(xy 113.03 41.91) (xy 116.84 41.91)
 		)
 		(stroke
@@
 	(wire
 		(pts
-			(xy 101.6 35.56) (xy 109.22 35.56)
+			(xy 105.41 41.91) (xy 113.03 41.91)
 		)
 		(stroke
@@
 	(wire
 		(pts
-			(xy 128.27 30.48) (xy 134.62 30.48)
+			(xy 132.08 36.83) (xy 138.43 36.83)
 		)
 		(stroke
@@
 	(wire
 		(pts
-			(xy 113.03 30.48) (xy 100.33 30.48)
+			(xy 116.84 36.83) (xy 104.14 36.83)
 		)
 		(stroke
@@
 	(wire
 		(pts
-			(xy 134.62 38.1) (xy 134.62 41.91)
+			(xy 138.43 44.45) (xy 138.43 48.26)
 		)
 		(stroke
@@
 	(wire
 		(pts
-			(xy 100.33 44.45) (xy 109.22 44.45)
+			(xy 104.14 50.8) (xy 113.03 50.8)
 		)
 		(stroke
@@
 	(wire
 		(pts
-			(xy 130.81 38.1) (xy 134.62 38.1)
+			(xy 134.62 44.45) (xy 138.43 44.45)
 		)
 		(stroke
@@
 	)
 	(label "HSE_OUT"
-		(at 143.51 30.48 180)
+		(at 147.32 36.83 180)
 		(effects
 			(font
@@
 	)
 	(label "HSE_IN"
-		(at 101.6 35.56 0)
+		(at 105.41 41.91 0)
 		(effects
 			(font
@@
 	(symbol
 		(lib_id "easyeda2kicad:X322525MOB4SI")
-		(at 120.65 33.02 0)
+		(at 124.46 39.37 0)
 		(unit 1)
 		(body_style 1)
@@
 		(fields_autoplaced yes)
 		(property "Reference" "X1"
-			(at 120.65 22.86 0)
+			(at 124.46 29.21 0)
 			(show_name no)
 			(do_not_autoplace no)
@@
 		)
 		(property "Value" "X322525MOB4SI"
-			(at 120.65 25.4 0)
+			(at 124.46 31.75 0)
 			(show_name no)
 			(do_not_autoplace no)
@@
 		)
 		(property "Footprint" "easyeda2kicad:CRYSTAL-SMD_4P-L3.2-W2.5-BL"
-			(at 120.65 43.18 0)
+			(at 124.46 49.53 0)
 			(hide yes)
 			(show_name no)
@@
 		)
 		(property "Datasheet" "https://lcsc.com/product-detail/SMD-Crystals_YSX321SL-25MHZ-12PF-10PPM-40-85_C9006.html"
-			(at 120.65 45.72 0)
+			(at 124.46 52.07 0)
 			(hide yes)
 			(show_name no)
@@
 		)
 		(property "Description" "YSX321SL 25MHZ 12PF 10PPM -40~+85℃"
-			(at 120.65 33.02 0)
+			(at 124.46 39.37 0)
 			(hide yes)
 			(show_name no)
@@
 		)
 		(property "Manufacturer" "YXC(扬兴晶振)"
-			(at 120.65 48.26 0)
+			(at 124.46 54.61 0)
 			(hide yes)
 			(show_name no)
@@
 		)
 		(property "MPN" "X322525MOB4SI"
-			(at 120.65 50.8 0)
+			(at 124.46 57.15 0)
 			(hide yes)
 			(show_name no)
@@
 		)
 		(property "LCSC Part" "C9006"
-			(at 120.65 53.34 0)
+			(at 124.46 59.69 0)
 			(hide yes)
 			(show_name no)
@@
 	(symbol
 		(lib_id "power:GND")
-		(at 134.62 41.91 0)
+		(at 138.43 48.26 0)
 		(unit 1)
 		(body_style 1)
@@
 		(fields_autoplaced yes)
 		(property "Reference" "#PWR043"
-			(at 134.62 48.26 0)
+			(at 138.43 54.61 0)
 			(hide yes)
 			(show_name no)
@@
 		)
 		(property "Value" "GND"
-			(at 134.62 46.99 0)
+			(at 138.43 53.34 0)
 			(show_name no)
 			(do_not_autoplace no)
@@
 		)
 		(property "Footprint" ""
-			(at 134.62 41.91 0)
+			(at 138.43 48.26 0)
 			(hide yes)
 			(show_name no)
@@
 		)
 		(property "Datasheet" ""
-			(at 134.62 41.91 0)
+			(at 138.43 48.26 0)
 			(hide yes)
 			(show_name no)
@@
 		)
 		(property "Description" "Power symbol creates a global label with name \"GND\" , ground"
-			(at 134.62 41.91 0)
+			(at 138.43 48.26 0)
 			(hide yes)
 			(show_name no)
@@
 	(symbol
 		(lib_id "Device:C")
-		(at 109.22 39.37 0)
+		(at 113.03 45.72 0)
 		(unit 1)
 		(body_style 1)
@@
 		(dnp no)
 		(property "Reference" "C33"
-			(at 104.902 37.338 0)
+			(at 108.712 43.688 0)
 			(show_name no)
 			(do_not_autoplace no)
@@
 		)
 		(property "Value" "20pF"
-			(at 103.632 41.91 0)
+			(at 107.442 48.26 0)
 			(show_name no)
 			(do_not_autoplace no)
@@
 		)
 		(property "Footprint" "Capacitor_SMD:C_0201_0603Metric"
-			(at 110.1852 43.18 0)
+			(at 113.9952 49.53 0)
 			(hide yes)
 			(show_name no)
@@
 		)
 		(property "Datasheet" ""
-			(at 109.22 39.37 0)
+			(at 113.03 45.72 0)
 			(hide yes)
 			(show_name no)
@@
 		)
 		(property "Description" "Unpolarized capacitor"
-			(at 109.22 39.37 0)
+			(at 113.03 45.72 0)
 			(hide yes)
 			(show_name no)
@@
 	(symbol
 		(lib_id "Device:C")
-		(at 134.62 34.29 0)
+		(at 138.43 40.64 0)
 		(unit 1)
 		(body_style 1)
@@
 		(fields_autoplaced yes)
 		(property "Reference" "C34"
-			(at 138.43 33.0199 0)
+			(at 142.24 39.3699 0)
 			(show_name no)
 			(do_not_autoplace no)
@@
 		)
 		(property "Value" "20pF"
-			(at 138.43 35.5599 0)
+			(at 142.24 41.9099 0)
 			(show_name no)
 			(do_not_autoplace no)
@@
 		)
 		(property "Footprint" "Capacitor_SMD:C_0201_0603Metric"
-			(at 135.5852 38.1 0)
+			(at 139.3952 44.45 0)
 			(hide yes)
 			(show_name no)
@@
 		)
 		(property "Datasheet" ""
-			(at 134.62 34.29 0)
+			(at 138.43 40.64 0)
 			(hide yes)
 			(show_name no)
@@
 		)
 		(property "Description" "Unpolarized capacitor"
-			(at 134.62 34.29 0)
+			(at 138.43 40.64 0)
 			(hide yes)
 			(show_name no)
@@
 	(symbol
 		(lib_id "power:GND")
-		(at 109.22 44.45 0)
+		(at 113.03 50.8 0)
 		(unit 1)
 		(body_style 1)
@@
 		(fields_autoplaced yes)
 		(property "Reference" "#PWR044"
-			(at 109.22 50.8 0)
+			(at 113.03 57.15 0)
 			(hide yes)
 			(show_name no)
@@
 		)
 		(property "Value" "GND"
-			(at 109.22 49.53 0)
+			(at 113.03 55.88 0)
 			(show_name no)
 			(do_not_autoplace no)
@@
 		)
 		(property "Footprint" ""
-			(at 109.22 44.45 0)
+			(at 113.03 50.8 0)
 			(hide yes)
 			(show_name no)
@@
 		)
 		(property "Datasheet" ""
-			(at 109.22 44.45 0)
+			(at 113.03 50.8 0)
 			(hide yes)
 			(show_name no)
@@
 		)
 		(property "Description" "Power symbol creates a global label with name \"GND\" , ground"
-			(at 109.22 44.45 0)
+			(at 113.03 50.8 0)
 			(hide yes)
 			(show_name no)

Commit message: Design Fixes
Parts:
- added R24: 52.3K, Resistor_SMD:R_0201_0603Metric, symbol Device:R
- added R25: 10K, Resistor_SMD:R_0201_0603Metric, symbol Device:R
Connections:
- net +5V: now also R13.1, R24.2; no longer R13.2, U5.5 (FB)
- net GND: now also R25.2
- net at U5.2 (PG): now also R13.2; no longer R13.1
- new net: R24.1, R25.1, U5.5 (FB)
Other:
- note added: "Changed CSB -> GND to CSB -> 3.3V CSB Tied to ground sets the sensor in SPI mode, while 3.3v selects I2C mode"
- note added: "Replaced the direct FB-to-VOUT connection on U5 (TPS63070RNMR) with a resistor divider to properly set the 5V output on this adjustable-variant part: R24 (52.3KΩ) between VOUT and FB, R25 (10KΩ) between FB and GND. The direct FB-VOUT tie was copied from a fixed-voltage-variant (TPS630701) app note and caused the regulator to servo down to its bare 0.8V internal reference instead of 5V."
- moved on the sheet: C10, C11, C12, C13, L4, R13
