File: hardware/Multipurpose Flight Computer.kicad_pcb (KiCad board)
At the start: 4 copper layers, 35 x 44.3 mm, 83 parts, among them J2 Conn_01x03, J3 Conn_01x03, J4 Conn_01x02_Pin, SW1 TS-1088-AR02016, SW2 TS-1088-AR02016, U1 BQ25883RGER, U2 ICM-45686, U3 STM32F722RETx, U4 BMP580, U5 TPS63070RNMR, U6 LMR51430, U7 TPD4EUSB30, X1 X322525MOB4SI

Commit message: Design Fixes
Parts:
- added R24: 52.3K, Resistor_SMD:R_0201_0603Metric, F.Cu at (145.3, 140.4)
- added R25: 10K, Resistor_SMD:R_0201_0603Metric, F.Cu at (144.2, 140.8)
- moved C13 1.27 mm to (144.8, 143.2)
- moved C12 0.82 mm to (150.9, 142.7)
- moved C10 0.77 mm to (148.9, 142.7)
- moved C11 0.77 mm to (146.9, 142.7)
- turned R13 to 0 degrees
Connections:
- R13 pad 1: Net-(U5-PG) -> +5V
- R13 pad 2: +5V -> Net-(U5-PG)
- U5 pad 5: +5V -> Net-(U5-FB)
Routing:
- net Net-(U5-FB): track 0.00 -> 1.88 mm
- net GND: track 125.2 -> 126.5 mm
- net +5V: track 18.5 -> 18.4 mm, vias 0 -> 2
